File: electronics/keyboard_controller/keyboard_controller.kicad_pcb (KiCad board)
At the start: 2 copper layers, 57 parts, among them J1 Conn_02x11_Odd_Even, J2 AVR-ISP-6, J3 Conn_01x02_Male, J4 Conn_01x03_Male, P1 USB_C_Plug_USB2.0, Q1 Q_NMOS_DGS, Q2 Q_NMOS_DGS, Q3 Q_PMOS_DGS, Q4 Q_NMOS_DGS, Q5 Q_PMOS_DGS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

Commit message: Worked on Placement
Parts:
- moved P1 104.9 mm to (87.6, 177.8), turned to 270 degrees
- moved R11 79.7 mm to (188.2, 80.0)
- moved R7 79.4 mm to (181.9, 80.0)
- moved R17 76.4 mm to (182.0, 85.7)
- moved R22 74.6 mm to (131.4, 160.4), turned to 270 degrees
- moved D3 73.5 mm to (145.4, 161.7), turned to 90 degrees
- moved R21 73.3 mm to (141.0, 161.0), turned to 90 degrees
- moved D4 72.8 mm to (135.9, 159.8), turned to 90 degrees
- moved R3 66.3 mm to (81.7, 57.8), turned to 180 degrees
- moved R26 64.9 mm to (157.5, 182.2), turned to 90 degrees
- moved D1 63.9 mm to (147.6, 54.0)
- moved R9 63.7 mm to (175.5, 57.1)
- moved C7 62.8 mm to (127.0, 45.1)
- moved J4 62.5 mm to (86.4, 168.9), turned to 180 degrees
- moved R20 61.1 mm to (134.4, 184.2)
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
Commit message: Worked no keyboard controller layout
Parts:
- J1: footprint Connector_PinHeader_1.27mm:PinHeader_2x11_P1.27mm_Vertical_SMD -> Connector_PinHeader_1.27mm:PinHeader_2x11_P1.27mm_Vertical
- P1: footprint Connector_USB:USB3_A_Molex_48393-001 -> Connector_USB:USB_C_Receptacle_Amphenol_12401548E4-2A_CircularHoles; moved to B.Cu
- Y1: footprint Crystal:Crystal_SMD_HC49-SD_HandSoldering -> Crystal:Crystal_HC49-4H_Vertical
- moved P1 110.0 mm to (92.7, 67.9), turned to 90 degrees
- moved R16 61.0 mm to (175.5, 96.5)
- moved C9 41.1 mm to (90.2, 143.3), turned to 270 degrees
- moved C8 39.2 mm to (90.2, 148.4), turned to 90 degrees
- moved C1 37.0 mm to (107.3, 84.2), turned to 270 degrees
- moved R18 35.0 mm to (95.0, 143.5)
- moved U3 34.9 mm to (95.2, 147.3), turned to 270 degrees
- moved R1 33.5 mm to (108.6, 80.6)
- moved J3 31.1 mm to (85.7, 127.6)
- moved J2 29.9 mm to (100.3, 82.5), turned to 0 degrees
- moved C2 29.8 mm to (113.7, 59.1), turned to 180 degrees
- moved R3 25.6 mm to (106.3, 64.8)
- moved R2 25.1 mm to (106.3, 67.3)
- moved R4 24.3 mm to (128.3, 69.0), turned to 90 degrees
- moved Y1 23.8 mm to (120.7, 87.0), turned to 180 degrees
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Connections:
- J1 pad 1: /SHIFT_LED -> /PA0
- J1 pad 10: /PB4 -> /PB5
- J1 pad 11: /PA4 -> /PA5
- J1 pad 12: /PB5 -> /PB4
- J1 pad 13: /PA3 -> /PA6
- J1 pad 14: /PB6 -> /PB3
- J1 pad 15: /PA2 -> /PA7
- J1 pad 16: /PB7 -> /PB2
- J1 pad 17: /PA1 -> /PC2
- J1 pad 18: /PC0 -> /PB1
- J1 pad 19: /PA0 -> /SHIFT_LED
- J1 pad 2: /PB0 -> /PC1
- J1 pad 20: /PC1 -> /PB0
- J1 pad 3: /PC2 -> /PA1
- J1 pad 4: /PB1 -> /PC0
- J1 pad 5: /PA7 -> /PA2
- J1 pad 6: /PB2 -> /PB7
- J1 pad 7: /PA6 -> /PA3
- J1 pad 8: /PB3 -> /PB6
- J1 pad 9: /PA5 -> /PA4
Routing:
- net /PB2: track 0.00 -> 74.2 mm, vias 0 -> 2
- net /PB3: track 0.00 -> 70.3 mm, vias 0 -> 2
- net /PB5: track 0.00 -> 61.4 mm, vias 0 -> 2
- net /PB6: track 0.00 -> 59.7 mm, vias 0 -> 2
- net /PB4: track 0.00 -> 55.8 mm, vias 0 -> 2
- net /PB7: track 0.00 -> 55.1 mm, vias 0 -> 2
- net /PC0: track 0.00 -> 43.8 mm, vias 0 -> 2
- net /PB1: track 0.00 -> 37.9 mm
- net /PC1: track 0.00 -> 37.8 mm, vias 0 -> 2
- net /RESET: track 0.00 -> 26.4 mm
- net GND: track 0.00 -> 21.1 mm
- net /PA0: track 0.00 -> 17.7 mm
- net /PA1: track 0.00 -> 16.6 mm
- net /PA2: track 0.00 -> 15.5 mm
- net /PA7: track 0.00 -> 12.0 mm
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Other:
- net class Default: via_dia 0.8 -> 0.6; via_drill 0.4 -> 0.3
- net class Double added: clearance 0.2, trace_width 0.5, via_dia 0.6, via_drill 0.3
